File: simble-overdrive.kicad_pcb (KiCad board)
At the start: 2 copper layers, 48.3 x 69.9 mm, 51 parts, among them Q1 2N7000, Q2 2N7000, U1 TLC2272

Commit message: minor fixes
Parts:
- renumbered SENSIVITY to SENSUTIVITY
