File: simble-overdrive.sch (KiCad schematic (older format))
At the start: 51 parts, among them Q1 2N7000, Q2 2N7000, U1 TLC2272

Commit message: minor fixes
Parts:
- renumbered SENSIVITY1 to SENSUTIVITY1
Changed lines of the file:
@@
 $EndComp
 $Comp
-L Device:R_POT SENSIVITY1
+L Device:R_POT SENSUTIVITY1
 U 1 1 5F2FB26D
 P 4650 5500
-F 0 "SENSIVITY1" V 4535 5500 50  0000 C CNN
+F 0 "SENSUTIVITY1" V 4535 5500 50  0000 C CNN
 F 1 "A1M" V 4444 5500 50  0000 C CNN
 F 2 "potentiometers:16MM_B.MOUNT" H 4650 5500 50  0001 C CNN
